File: stabiljr.kicad_sch (KiCad schematic)
At the start: 17 parts, among them J1 Conn_01x24, J2 Conn_01x20, M1 Module-power_12and5V-0.2, M4 Module-vr-max9924-0.1

Commit message: TEST3
Parts:
- renumbered İŞLEMC1 to CPU1
Changed lines of the file:
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@@
 		(on_board yes)
 		(dnp no)
-		(property "Reference" "İŞLEMC1"
+		(property "Reference" "CPU1"
 			(at 214.376 89.916 0)
 			(effects
@@
 			(project "uaefi"
 				(path "/ac264c30-3e9a-4be2-b97a-9949b68bd497"
-					(reference "İŞLEMC1")
+					(reference "CPU1")
 					(unit 1)
 				)
@@
 		)
 		(instances
-			(project "stabildaytona"
+			(project "stabiljr"
 				(path "/ac264c30-3e9a-4be2-b97a-9949b68bd497"
 					(page "10")
@@
 		)
 		(instances
-			(project "stabildaytona"
+			(project "stabiljr"
 				(path "/ac264c30-3e9a-4be2-b97a-9949b68bd497"
 					(page "3")
@@
 		)
 		(instances
-			(project "stabildaytona"
+			(project "stabiljr"
 				(path "/ac264c30-3e9a-4be2-b97a-9949b68bd497"
 					(page "8")
@@
 		)
 		(instances
-			(project "stabildaytona"
+			(project "stabiljr"
 				(path "/ac264c30-3e9a-4be2-b97a-9949b68bd497"
 					(page "9")
@@
 		)
 		(instances
-			(project "stabildaytona"
+			(project "stabiljr"
 				(path "/ac264c30-3e9a-4be2-b97a-9949b68bd497"
 					(page "6")
@@
 		)
 		(instances
-			(project "stabildaytona"
+			(project "stabiljr"
 				(path "/ac264c30-3e9a-4be2-b97a-9949b68bd497"
 					(page "2")

Commit message: TEST4
Parts:
- R41, R42: LCSC C17414 -> ERA6AEB272V
Changed lines of the file:
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@@
 			)
 		)
-		(property "LCSC" "C17414"
+		(property "LCSC" "ERA6AEB272V"
 			(at 151.13 186.69 0)
 			(effects
@@
 			)
 		)
-		(property "LCSC" "C17414"
+		(property "LCSC" "ERA6AEB272V"
 			(at 151.13 182.88 0)
 			(effects

Commit message: test5
Parts:
- R43: value 10K -> 10k
Changed lines of the file:
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@@
 			)
 		)
-		(property "Value" "10K"
+		(property "Value" "10k"
 			(at 146.05 193.04 0)
 			(effects
