File: stabiljr.kicad_pcb (KiCad board)
At the start: 4 copper layers, 98.5 x 110 mm, 42 parts, among them J1 Conn_01x24, J2 Conn_01x20, M1 Module-power_12and5V-0.2, M4 Module-vr-max9924-0.1, U1 VNLD5160TR-E, U10 VNLD5160TR-E, U2 VNLD5160TR-E, U3 VNLD5160TR-E, U9 VNLD5160TR-E

Commit message: TEST3
Parts:
- removed İŞLEMC1: Module:mega-mcu100/0.3, hellen-one-mega-mcu100-0.3:mega-mcu100
- added CPU1: Module:mega-mcu100/0.3, hellen-one-mega-mcu100-0.3:mega-mcu100, F.Cu at (92.8, 63.1)

Commit message: ok
Other:
- board text added: "1"
- board text added: "20"
Changed lines of the file:
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@@
 			(pintype "passive+no_connect")
 		)
-		(model ":hellen-one-models:MPXH6400A.STEP"
+		(model "${KIPRJMOD}/kicad6-libraries/MPXH6400A.STEP"
 			(offset
 				(xyz -6 7.7 6.3)
@@
 			)
 		)
+		(model "${KIPRJMOD}/hellen-one/modules/vr-max9924/0.3/vr-max9924-vrml.wrl"
+			(offset
+				(xyz 0 0 -0.8)
+			)
+			(scale
+				(xyz 0.4 0.4 0.15)
+			)
+			(rotate
+				(xyz 0 0 0)
+			)
+		)
 	)
 	(footprint "Connector_JST:JST_PH_B4B-PH-K_1x04_P2.00mm_Vertical"
@@
 				(font
 					(size 0.6 0.6)
-					(thickness 0.254)
+					(thickness 0.15)
 				)
 				(justify left bottom)
@@
 				(font
 					(size 0.6 0.6)
-					(thickness 0.254)
+					(thickness 0.15)
 				)
 				(justify left bottom)
@@
 			)
 		)
+		(model "${KIPRJMOD}/hellen-one/modules/power_12and5V/0.3/power_12and5V-vrml.wrl"
+			(offset
+				(xyz 0 0 -0.15)
+			)
+			(scale
+				(xyz 0.4 0.4 0.33)
+			)
+			(rotate
+				(xyz 0 0 0)
+			)
+		)
 	)
 	(footprint "hellen-one-common:R0603"
@@
 			)
 		)
-		(model "${KIPRJMOD}/EASYEDA_MODELS/CONN-TH_HCCPHPE24BKA90F.step"
+		(model "C:/Users/OZER/Desktop/3d/HCCPHPE24BKA90F v10.step"
 			(offset
-				(xyz 33.0999 0.8 -4)
+				(xyz -33 -19 10.5)
 			)
 			(scale
@@
 			)
 			(rotate
-				(xyz -0 -0 0)
+				(xyz 90 180 -180)
 			)
 		)
@@
 			)
 		)
+		(model "${KIPRJMOD}/hellen-one/modules/mega-mcu100/0.3/mega-mcu100-vrml.wrl"
+			(offset
+				(xyz 0 0 -0.1)
+			)
+			(scale
+				(xyz 0.4 0.4 0.35)
+			)
+			(rotate
+				(xyz 0 0 0)
+			)
+		)
 	)
 	(footprint "hellen-one-common:R0603"
@@
 		)
 		(model "${KICAD8_3DMODEL_DIR}/Package_SO.3dshapes/SOIC-8_3.9x4.9mm_P1.27mm.wrl"
+			(hide yes)
 			(offset
 				(xyz 0 0 0)
@@
 			)
 		)
+		(model "${KIPRJMOD}/hellen-one/kicad/models/SOIC08 narrow.STEP"
+			(offset
+				(xyz 0 0 0)
+			)
+			(scale
+				(xyz 1 1 1)
+			)
+			(rotate
+				(xyz 0 0 90)
+			)
+		)
 	)
 	(footprint "Fuse:Fuse_0603_1608Metric"
@@
 		(layer "Edge.Cuts")
 	)
+	(gr_text "1"
+		(at 72 46 0)
+		(layer "F.SilkS")
+		(effects
+			(font
+				(size 1 1)
+				(thickness 0.15)
+			)
+			(justify left bottom)
+		)
+	)
+	(gr_text "20"
+		(at 147 45.5 0)
+		(layer "F.SilkS")
+		(effects
+			(font
+				(size 1 1)
+				(thickness 0.15)
+			)
+			(justify left bottom)
+		)
+	)
 	(gr_text "ÖZER"
